Commit message: stance mode worked

File: legged_examples/legged_hunter/legged_hunter_description/urdf/hunter_sim.urdf (robot description, URDF)
Before this commit: robot hunter, 16 links, 15 joints
Links:
- link base_link: mass 5.673631 -> 1.6042619; geometry collision box size=0.1 0.1 0.09; visual mesh filename=package://legged_hunter_description/meshes_pi/base_link.STL
- link leg_l1_link: mass 0.453728 -> 0.12545; geometry collision box size=0.0001 0.0001 0.0001; visual mesh filename=package://legged_hunter_description/meshes_pi/leg_l1_link.S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
- link leg_l2_link: mass 0.925998 -> 0.34; geometry collision box size=0.0001 0.0001 0.0001; visual mesh filename=package://legged_hunter_description/meshes_pi/leg_l2_link.S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
- link leg_l3_link: mass 1.390468 -> 0.476; geometry collision box size=0.01 0.01 0.09; visual mesh filename=package://legged_hunter_description/meshes_pi/leg_l3_link.S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
- link leg_l4_link: mass 0.649518 -> 0.361; geometry collision box size=0.01 0.01 0.09; visual mesh filename=package://legged_hunter_description/meshes_pi/leg_l4_link.S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
- link leg_l5_link: mass 0.030265 -> 0.089; geometry collision box size=0.1 0.04 0.01; visual box size=0.1 0.04 0.01
- link leg_r1_link: mass 0.453728 -> 0.367; geometry collision box size=0.0001 0.0001 0.0001; visual mesh filename=package://legged_hunter_description/meshes_pi/leg_r1_link.S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
- link leg_r2_link: mass 0.925998 -> 0.34; geometry collision box size=0.0001 0.0001 0.0001; visual mesh filename=package://legged_hunter_description/meshes_pi/leg_r2_link.S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
- link leg_r3_link: mass 1.388625 -> 0.476; geometry collision box size=0.01 0.01 0.09; visual mesh filename=package://legged_hunter_description/meshes_pi/leg_r3_link.S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
- link leg_r4_link: mass 0.614720 -> 0.361; geometry collision box size=0.01 0.01 0.09; visual mesh filename=package://legged_hunter_description/meshes_pi/leg_r4_link.S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
- link leg_r5_link: mass 0.030265 -> 0.089; geometry collision box size=0.1 0.04 0.01; visual box size=0.1 0.04 0.01
Joints:
- joint leg_l1_joint: axis 1 0 0 -> 0 0 1; limit lower=-0.2 upper=0.5 effort=23.7 velocity=30.1 -> lower=-1.0 upper=1.0 effort=15 velocity=20; origin xyz=-0.002 0.09 -0.1035 rpy=0 0 0 -> xyz=0 0 0.054 rpy=-1.5708 0 1.5708; parent base_link -> leg_l2_link
- joint leg_l2_joint: limit lower=-0.5 upper=1 effort=23.7 velocity=30.1 -> lower=-1.0 upper=1.0 effort=15 velocity=20; origin xyz=0 -0.00016972 -0.0325 rpy=0 0 0 -> xyz=0 0.045 0 rpy=-3.1416 0 -3.1416; parent leg_l1_link -> base_link
- joint leg_l3_joint: axis 0 -1 0 -> 0 0 1; limit lower=-0.8 upper=1.2 effort=23.7 velocity=30.1 -> lower=-0.7854 upper=1.15 effort=15 velocity=20; origin xyz=0 -0.01433 -0.0575 rpy=0 0 0 -> xyz=0 0 0.002 rpy=1.5708 0 -1.5708; parent leg_l2_link -> leg_l1_link
- joint leg_l4_joint: axis 0 1 0 -> 0 0 1; limit lower=0 upper=1.5 effort=23.7 velocity=30.1 -> lower=0 upper=1.5 effort=15 velocity=20; origin xyz=0 0.0145 -0.24 rpy=0 0 0 -> xyz=0.15 0 0 rpy=3.1416 0 0
- joint leg_l5_joint: axis 0 -1 0 -> 0 0 1; limit lower=-1.1 upper=1.1 effort=23.7 velocity=30.1 -> lower=-0.75 upper=0.75 effort=15 velocity=20; origin xyz=0.005 0 -0.23995 rpy=0 0 0 -> xyz=0.16 0 0 rpy=3.1416 0 -1.5708
- joint leg_r1_joint: axis 1 0 0 -> 0 0 1; limit lower=-0.5 upper=0.2 effort=23.7 velocity=30.1 -> lower=-1.0 upper=1.0 effort=15 velocity=20; origin xyz=-0.002 -0.09 -0.1035 rpy=0 0 0 -> xyz=0 0 0.054 rpy=1.5708 0 0; parent base_link -> leg_r2_link
- joint leg_r2_joint: axis 0 0 1 -> 0 0 -1; limit lower=-1 upper=0.5 effort=23.7 velocity=30.1 -> lower=-1.0 upper=1.0 effort=15 velocity=20; origin xyz=0 0.00016972 -0.0325 rpy=0 0 0 -> xyz=0 -0.045 0 rpy=3.1416 0 -1.5708; parent leg_r1_link -> base_link
- joint leg_r3_joint: axis 0 1 0 -> 0 0 1; limit lower=-1.2 upper=0.8 effort=23.7 velocity=30.1 -> lower=-1.15 upper=0.7854 effort=15 velocity=21; origin xyz=0 0.01633 -0.0575 rpy=0 0 0 -> xyz=0 0 0.002 rpy=-1.5708 0 1.5708; parent leg_r2_link -> leg_r1_link
- joint leg_r4_joint: axis 0 1 0 -> 0 0 1; limit lower=0 upper=1.5 effort=23.7 velocity=30.1 -> lower=-1.5 upper=0.0 effort=15 velocity=20; origin xyz=0 -0.0145 -0.24 rpy=0 0 0 -> xyz=0.15 0 0 rpy=-3.1416 0 0
- joint leg_r5_joint: axis 0 1 0 -> 0 0 1; limit lower=-1.1 upper=1.1 effort=23.7 velocity=30.1 -> lower=-0.75 upper=0.75 effort=15 velocity=20; origin xyz=0.005 0 -0.23995 rpy=0 0 0 -> xyz=0.16 0 0 rpy=3.1416 0 1.5708
