Commit message: change distance between two legs
fix stand state

File: legged_examples/legged_hunter/legged_hunter_description/urdf/hunter.urdf (robot description, URDF)
Before this commit: robot hunter, 16 links, 15 joints
Joints:
- joint leg_l1_joint: limit lower=-1.0 upper=1.0 effort=15 velocity=20 -> lower=-0.2 upper=0.5 effort=15 velocity=20
- joint leg_l2_joint: axis 0 0 1 -> 0 0 -1; limit lower=-1.0 upper=1.0 effort=15 velocity=20 -> lower=-0.5 upper=1 effort=15 velocity=20; origin xyz=0 0.045 0 rpy=-3.1416 0 -3.1416 -> xyz=0 0.075 0 rpy=-3.1416 0 -3.1416
- joint leg_l3_joint: limit lower=-0.7854 upper=1.15 effort=15 velocity=20 -> lower=-0.8 upper=1.2 effort=15 velocity=20
- joint leg_l5_joint: limit lower=-0.75 upper=0.75 effort=15 velocity=20 -> lower=-1.1 upper=1.1 effort=15 velocity=20
- joint leg_r1_joint: limit lower=-1.0 upper=1.0 effort=15 velocity=20 -> lower=-0.5 upper=0.2 effort=15 velocity=20
- joint leg_r2_joint: limit lower=-1.0 upper=1.0 effort=15 velocity=20 -> lower=-1 upper=0.5 effort=15 velocity=20; origin xyz=0 -0.045 0 rpy=3.1416 0 -1.5708 -> xyz=0 -0.075 0 rpy=3.1416 0 -1.5708
- joint leg_r3_joint: limit lower=-1.15 upper=0.7854 effort=15 velocity=21 -> lower=-1.2 upper=0.8 effort=15 velocity=21
- joint leg_r4_joint: axis 0 0 1 -> 0 0 -1; limit lower=-1.5 upper=0.0 effort=15 velocity=20 -> lower=0 upper=1.5 effort=15 velocity=20
- joint leg_r5_joint: limit lower=-0.75 upper=0.75 effort=15 velocity=20 -> lower=-1.1 upper=1.1 effort=15 velocity=20

File: legged_examples/legged_hunter/legged_hunter_description/urdf/source/hunter.urdf (robot description, URDF)
Before this commit: robot hunter, 16 links, 15 joints
Links:
- link base_link: geometry collision box size=0.184 0.15 0.2; visual mesh filename=/home/sunteng/control_ws/src/hunter_bipedal_control/legged_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
- link leg_l1_link: geometry collision box size=0.06 0.07 0.155; visual mesh filename=/home/sunteng/control_ws/src/hunter_bipedal_control/legged_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
- link leg_l2_link: geometry collision cylinder length=0.146 radius=0.065; visual mesh filename=/home/sunteng/control_ws/src/hunter_bipedal_control/legged_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
- link leg_l3_link: geometry collision box size=0.06 0.25 0.05; visual mesh filename=/home/sunteng/control_ws/src/hunter_bipedal_control/legged_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
- link leg_l4_link: geometry collision box size=0.041 0.25 0.03; collision cylinder length=0.07 radius=0.034
- link leg_l5_link: geometry collision box size=0.1001 0.0345 0.0175; visual mesh filename=/home/sunteng/control_ws/src/hunter_bipedal_control/legged_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
- link leg_r1_link: geometry collision box size=0.06 0.07 0.155; visual mesh filename=/home/sunteng/control_ws/src/hunter_bipedal_control/legged_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
- link leg_r2_link: geometry collision cylinder length=0.146 radius=0.065; visual mesh filename=/home/sunteng/control_ws/src/hunter_bipedal_control/legged_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
- link leg_r3_link: geometry collision box size=0.06 0.25 0.05; visual mesh filename=/home/sunteng/control_ws/src/hunter_bipedal_control/legged_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
- link leg_r4_link: geometry collision box size=0.041 0.25 0.03; collision cylinder length=0.07 radius=0.034
- link leg_r5_link: geometry collision box size=0.1001 0.0345 0.0175; visual mesh filename=/home/sunteng/control_ws/src/hunter_bipedal_control/legged_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

File: legged_examples/legged_hunter/legged_hunter_description/urdf/source/hunter_sim.urdf (robot description, URDF)
Before this commit: robot hunter, 16 links, 15 joints
Links:
- link base_link: geometry collision box size=0.184 0.15 0.2; visual mesh filename=/home/sunteng/control_ws/src/hunter_bipedal_control/legged_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
- link leg_l1_link: geometry collision box size=0.06 0.07 0.155; visual mesh filename=/home/sunteng/control_ws/src/hunter_bipedal_control/legged_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
- link leg_l2_link: geometry collision cylinder length=0.146 radius=0.065; visual mesh filename=/home/sunteng/control_ws/src/hunter_bipedal_control/legged_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
- link leg_l3_link: geometry collision box size=0.06 0.25 0.05; visual mesh filename=/home/sunteng/control_ws/src/hunter_bipedal_control/legged_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
- link leg_l4_link: geometry collision box size=0.041 0.25 0.03; collision cylinder length=0.07 radius=0.034
- link leg_l5_link: geometry collision box size=0.1001 0.0345 0.0175; visual mesh filename=/home/sunteng/control_ws/src/hunter_bipedal_control/legged_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
- link leg_r1_link: geometry collision box size=0.06 0.07 0.155; visual mesh filename=/home/sunteng/control_ws/src/hunter_bipedal_control/legged_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
- link leg_r2_link: geometry collision cylinder length=0.146 radius=0.065; visual mesh filename=/home/sunteng/control_ws/src/hunter_bipedal_control/legged_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
- link leg_r3_link: geometry collision box size=0.06 0.25 0.05; visual mesh filename=/home/sunteng/control_ws/src/hunter_bipedal_control/legged_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
- link leg_r4_link: geometry collision box size=0.041 0.25 0.03; collision cylinder length=0.07 radius=0.034
- link leg_r5_link: geometry collision box size=0.1001 0.0345 0.0175; visual mesh filename=/home/sunteng/control_ws/src/hunter_bipedal_control/legged_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

Commit message: fixed inertial in URDF, now it walks smoothly in Gazebo

File: legged_examples/legged_hunter/legged_hunter_description/urdf/hunter.urdf (robot description, URDF)
Before this commit: robot hunter, 16 links, 15 joints
Links:
- link base_link: geometry collision box size=0.1 0.1 0.09; visual mesh filename=package://legged_hunter_description/meshes/base_link.STL
- link leg_l1_link: mass 0.12545 -> 0.367; geometry collision box size=0.0001 0.0001 0.0001; visual mesh filename=package://legged_hunter_description/meshes/l_hip_roll_link.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
- link leg_l2_link: geometry collision box size=0.0001 0.0001 0.0001; visual mesh filename=package://legged_hunter_description/meshes/l_hip_yaw_link.S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
- link leg_l3_link: geometry collision box size=0.01 0.01 0.09; visual mesh filename=package://legged_hunter_description/meshes/l_thigh_link.STL
- link leg_l4_link: geometry collision box size=0.01 0.01 0.09; visual mesh filename=package://legged_hunter_description/meshes/l_calf_link.STL
- link leg_r1_link: geometry collision box size=0.0001 0.0001 0.0001; visual mesh filename=package://legged_hunter_description/meshes/r_hip_roll_link.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
- link leg_r2_link: geometry collision box size=0.0001 0.0001 0.0001; visual mesh filename=package://legged_hunter_description/meshes/r_hip_yaw_link.S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
- link leg_r3_link: geometry collision box size=0.01 0.01 0.09; visual mesh filename=package://legged_hunter_description/meshes/r_thigh_link.STL
- link leg_r4_link: geometry collision box size=0.01 0.01 0.09; visual mesh filename=package://legged_hunter_description/meshes/r_calf_link.STL
Joints:
- joint leg_l1_joint: axis 0 0 1 -> 1 0 0; limit lower=-0.2 upper=0.5 effort=15 velocity=20 -> lower=-3.14 upper=3.14 effort=21 velocity=21; origin xyz=0 0 0.054 rpy=-1.5708 0 1.5708 -> xyz=-0.037 0 -0.054 rpy=0 0 0
- joint leg_l2_joint: axis 0 0 -1 -> 0 0 1; limit lower=-0.5 upper=1 effort=15 velocity=20 -> lower=-3.14 upper=3.14 effort=21 velocity=21; origin xyz=0 0.075 0 rpy=-3.1416 0 -3.1416 -> xyz=0 0.075 0 rpy=0 0 0
- joint leg_l3_joint: axis 0 0 1 -> 0 -1 0; limit lower=-0.8 upper=1.2 effort=15 velocity=20 -> lower=-3.14 upper=3.14 effort=21 velocity=21; origin xyz=0 0 0.002 rpy=1.5708 0 -1.5708 -> xyz=0.039 0 0 rpy=0 0 0
- joint leg_l4_joint: axis 0 0 1 -> 0 1 0; limit lower=0 upper=1.5 effort=15 velocity=20 -> lower=-3.14 upper=3.14 effort=21 velocity=21; origin xyz=0.15 0 0 rpy=3.1416 0 0 -> xyz=0 0 -0.15 rpy=0 0 0
- joint leg_l5_joint: axis 0 0 1 -> 0 -1 0; limit lower=-1.1 upper=1.1 effort=15 velocity=20 -> lower=-3.14 upper=3.14 effort=21 velocity=21; origin xyz=0.16 0 0 rpy=3.1416 0 -1.5708 -> xyz=0 0 -0.16 rpy=0 0 0
- joint leg_r1_joint: axis 0 0 1 -> 1 0 0; limit lower=-0.5 upper=0.2 effort=15 velocity=20 -> lower=-3.14 upper=3.14 effort=21 velocity=21; origin xyz=0 0 0.054 rpy=1.5708 0 0 -> xyz=-0.037 0 -0.054 rpy=0 0 0
- joint leg_r2_joint: axis 0 0 -1 -> 0 0 1; limit lower=-1 upper=0.5 effort=15 velocity=20 -> lower=-3.14 upper=3.14 effort=21 velocity=21; origin xyz=0 -0.075 0 rpy=3.1416 0 -1.5708 -> xyz=0 -0.075 0 rpy=0 0 0
- joint leg_r3_joint: axis 0 0 1 -> 0 1 0; limit lower=-1.2 upper=0.8 effort=15 velocity=21 -> lower=-3.14 upper=3.14 effort=21 velocity=21; origin xyz=0 0 0.002 rpy=-1.5708 0 1.5708 -> xyz=0.039 0 0 rpy=0 0 0
- joint leg_r4_joint: axis 0 0 -1 -> 0 1 0; limit lower=0 upper=1.5 effort=15 velocity=20 -> lower=-3.14 upper=3.14 effort=21 velocity=21; origin xyz=0.15 0 0 rpy=-3.1416 0 0 -> xyz=0 0 -0.15 rpy=0 0 0
- joint leg_r5_joint: axis 0 0 1 -> 0 1 0; limit lower=-1.1 upper=1.1 effort=15 velocity=20 -> lower=-3.14 upper=3.14 effort=21 velocity=21; origin xyz=0.16 0 0 rpy=3.1416 0 1.5708 -> xyz=0 0 -0.16 rpy=0 0 0
